Commit message: Submitting changes made to syndey world

File: extra/vrx_gazebo tweaks/world files to place in vrx_gazebo worlds folder/tasks.world.xacro (robot description, xacro)
@@ -88,44 +88,4 @@
       <uri>model://turtle_buoy</uri>
     </include>
-    <!-- The scoring plugin -->
-    <plugin name="wildlife_scoring_plugin"
-            filename="libwildlife_scoring_plugin.so">
-      <!-- Common parameters -->
-      <vehicle>wamv</vehicle>
-      <task_name>wildlife</task_name>
-      <initial_state_duration>10</initial_state_duration>
-      <ready_state_duration>10</ready_state_duration>
-      <running_state_duration>300</running_state_duration>
-      <collision_buffer>10</collision_buffer>
-      <release_joints>
-        <joint>
-          <name>wamv_external_pivot_joint</name>
-        </joint>
-        <joint>
-          <name>wamv_external_riser</name>
-        </joint>
-      </release_joints>
-      <!-- wildlife specific parameters -->
-      <buoys>
-        <buoy>
-          <model_name>crocodile_buoy</model_name>
-          <link_name>link</link_name>
-          <goal>avoid</goal>
-        </buoy>
-        <buoy>
-          <model_name>platypus_buoy</model_name>
-          <link_name>link</link_name>
-          <goal>circumnavigate_clockwise</goal>
-        </buoy>
-        <buoy>
-          <model_name>turtle_buoy</model_name>
-          <link_name>link</link_name>
-          <goal>circumnavigate_counterclockwise</goal>
-        </buoy>
-      </buoys>
-      <engagement_distance>10.0</engagement_distance>
-      <time_bonus>30.0</time_bonus>
-      <animals_topic>/vrx/wildlife/animals/poses</animals_topic>
-    </plugin>
     <!-- MC = Task 5-->
     <!-- The light buoy -->
